Commit message: 修复夹抓抓取bug

File: src/robot_arm/urdf/robot_arm.urdf (robot description, URDF)
Before this commit: robot robot_arm, 9 links, 8 joints
Joints:
- joint joint3: limit lower=-1.2 upper=4.4 effort=0 velocity=0.3142 -> lower=-1.2 upper=1.5708 effort=0 velocity=0.3142
- joint joint4: limit lower=-3.1 upper=3.1 effort=0 velocity=0.4887 -> lower=-3.1416 upper=3.1416 effort=0 velocity=0.4887
- joint joint6: limit lower=-6.284 upper=6.284 effort=0 velocity=0.4887 -> lower=-6.283 upper=6.283 effort=0 velocity=0.4887

Commit message: 修复bug，增加机械臂位置反馈

File: src/robot_arm/urdf/robot_arm.urdf (robot description, URDF)
Before this commit: robot robot_arm, 9 links, 8 joints
Joints:
- joint joint6: limit lower=-6.283 upper=6.283 effort=0 velocity=0.4887 -> lower=-3.15 upper=3.15 effort=0 velocity=0.4887

Commit message: 稳定版

File: src/robot_arm/urdf/robot_arm.urdf (robot description, URDF)
Before this commit: robot robot_arm, 9 links, 8 joints
Joints:
- joint joint4: limit lower=-3.1416 upper=3.1416 effort=0 velocity=0.4887 -> lower=-3.14 upper=3.14 effort=0 velocity=0.4887
- joint joint6: limit lower=-3.15 upper=3.15 effort=0 velocity=0.4887 -> lower=-1.57 upper=1.57 effort=0 velocity=0.4887
